Commit message: [Update] update base_link

File: turtlebot3/turtlebot3_description/urdf/turtlebot3_waffle.urdf.xacro (robot description, xacro)
@@ -139,17 +139,17 @@
   <joint name="scan_joint" type="fixed">
     <parent link="base_link"/>
-    <child link="base_scan"/>
-    <origin xyz="-0.064 0 0.122" rpy="0 0 0"/>
-  </joint>
-  <link name="base_scan">
-    <visual>
-      <origin xyz="0 0 0" rpy="0 0 0"/>
-      <geometry>
-        <mesh filename="package://turtlebot3_description/meshes/sensors/lds.stl" scale="0.001 0.001 0.001"/>
+    <child link="laser"/>
+    <origin xyz="0.05 0 0.125" rpy="0 0 0"/>
+  </joint>
+  <link name="laser">
+    <visual>
+      <origin xyz="0 0 0.02" rpy="0 0 0"/>
+      <geometry>
+        <mesh filename="package://turtlebot3_description/meshes/sensors/urg_optical_axis_center_origin.dae"/>
       </geometry>
       <material name="dark"/>
     </visual>
     <collision>
-      <origin xyz="0.015 0 -0.0065" rpy="0 0 0"/>
+      <origin xyz="0 0 0" rpy="0 0 0"/>
       <geometry>
         <cylinder length="0.0315" radius="0.055"/>
@@ -157,12 +157,12 @@
     </collision>
     <inertial>
-      <mass value="0.114" />
-      <origin xyz="0 0 0" />
-      <inertia ixx="0.001" ixy="0.0" ixz="0.0"
-               iyy="0.001" iyz="0.0"
-               izz="0.001" />
-    </inertial>
-  </link>
-  <joint name="camera_joint" type="fixed">
+      <mass value="0.270" />
+      <origin xyz="0 0 0" />
+      <inertia ixx="2.632e-4" ixy="0.0" ixz="0.0"
+               iyy="2.632e-4" iyz="0.0"
+               izz="1.62e-4" />
+    </inertial>
+  </link>
+  <!-- <joint name="camera_joint" type="fixed">
     <origin xyz="0.064 -0.065 0.094" rpy="0 0 0"/>
     <parent link="base_link"/>
@@ -181,5 +181,5 @@
         <box size="0.012 0.132 0.020"/>
       </geometry>
-    </collision>
+    </collision> -->
     <!-- This inertial field needs doesn't contain reliable data!! -->
 <!--   <inertial>
@@ -190,6 +190,6 @@
                izz="0.003879257" />
     </inertial>-->
-  </link>
-  <joint name="camera_rgb_joint" type="fixed">
+  <!-- </link> -->
+  <!-- <joint name="camera_rgb_joint" type="fixed">
     <origin xyz="${r200_cam_rgb_px} ${r200_cam_rgb_py} ${r200_cam_rgb_pz}" rpy="0 0 0"/>
     <parent link="camera_link"/>
@@ -214,4 +214,4 @@
     <child link="camera_depth_optical_frame"/>
   </joint>
-  <link name="camera_depth_optical_frame"/>
+  <link name="camera_depth_optical_frame"/> -->
 </robot>

Commit message: [Update]

File: turtlebot3/turtlebot3_description/urdf/turtlebot3_waffle.urdf.xacro (robot description, xacro)
@@ -140,5 +140,5 @@
     <parent link="base_link"/>
     <child link="laser"/>
-    <origin xyz="0.05 0 0.125" rpy="0 0 0"/>
+    <origin xyz="0.02 0 0.125" rpy="0 0 0"/>
   </joint>
   <link name="laser">

Commit message: sensor_bridge

File: turtlebot3/turtlebot3_description/urdf/turtlebot3_waffle.urdf.xacro (robot description, xacro)
@@ -164,4 +164,19 @@
     </inertial>
   </link>
+<!-- T265 -->
+  <link name="camera_link">
+    <visual>
+      <origin xyz="0.02 0 0.02" rpy="0 0 0" />
+      <geometry>
+        <box size="0.05 0.19 0.005" />
+      </geometry>
+      <material name="blue" />
+    </visual>
+  </link>
+ <joint name="camera_joint" type="fixed">
+    <parent link="base_link" />
+    <child link="camera_link" />
+    <origin xyz="0.03 0 0.125" rpy="0 0 0" />
+  </joint>
   <!-- <joint name="camera_joint" type="fixed">
     <origin xyz="0.064 -0.065 0.094" rpy="0 0 0"/>

Commit message: [Update] update T265 odom to cartographer

File: turtlebot3/turtlebot3_description/urdf/turtlebot3_waffle.urdf.xacro (robot description, xacro)
@@ -165,5 +165,10 @@
   </link>
 <!-- T265 -->
-  <link name="camera_link">
+  <joint name="t265_joint" type="fixed">
+    <parent link="base_link" />
+    <child link="t265_link" />
+    <origin xyz="0.03 0 0.125" rpy="0 0 0" />
+  </joint>
+  <link name="t265_link">
     <visual>
       <origin xyz="0.02 0 0.02" rpy="0 0 0" />
@@ -174,9 +179,4 @@
     </visual>
   </link>
- <joint name="camera_joint" type="fixed">
-    <parent link="base_link" />
-    <child link="camera_link" />
-    <origin xyz="0.03 0 0.125" rpy="0 0 0" />
-  </joint>
   <!-- <joint name="camera_joint" type="fixed">
     <origin xyz="0.064 -0.065 0.094" rpy="0 0 0"/>
